Commit message: Updated Heatmap Logic

File: capstone_ws/src/bee_farm_sim/bee_farm_sim/description/cube_bot.xacro (robot description, xacro)
@@ -5,5 +5,5 @@
     <visual>
       <geometry>
-        <box size="0.5 0.5 0.5"/>
+        <box size="0.2 0.2 0.2"/>
       </geometry>
       <material name="black">
@@ -14,5 +14,5 @@
     <collision>
       <geometry>
-        <box size="0.5 0.5 0.5"/>
+        <box size="0.2 0.2 0.2"/>
       </geometry>
     </collision>
